File: NxtPX4.kicad_sch (KiCad schematic)
At the start: 147 parts, among them J1 USB_C_Receptacle_USB2.0, J10 ESC, J23 Conn_01x04, J24 Conn_01x02_Pin, J24 Micro_SD_Card, J25 Conn_01x02_Pin, J26 Conn_01x02_Pin, J27 GND, J4 ESC, J6 ESC, J8 UART_Combo, J9 Upper computer connector, Q1 AP40P05, Q2 SS8050(NPN BEC), Q3 SS8050(NPN BEC), U10 BMI088, U11 ICM-20602, U12 HiLAB_Logo, U13 BMP388, U14 W25Q128JVS, U15 Signature, U16 High_temp, U17 high_voltage, U18 Caution, U2 RT9013-33GB, U22 ICM-42688-P, U23 MPU6500/ICM20649, U3 RT9013-33GB, U5 HKU_Logo, U6 UAV_LOGO, U7 Direction_Logo, U8 RI_LOGO, U9 STM32H743VIH6, Y1 SG-210STF/ X1G004171002700, Y2 ABS07 (32.768kHZ)

Commit message: Latest Update
Parts:
- removed C40, C53, C54, C55: 100nF(0201 10V 10%), Capacitor_SMD:C_0201_0603Metric, symbol Device:C_Small
- removed C41: 2.2uF(0201 10V 10%), Capacitor_SMD:C_0201_0603Metric, symbol Device:C_Small
- removed C43: 10nF(0201 10V 10%), Capacitor_SMD:C_0201_0603Metric, symbol Device:C_Small
- removed C46: 100nF(0201 10V), Capacitor_SMD:C_0201_0603Metric, symbol Device:C_Small
- removed D11: LED_Blue(0201), LED_SMD:LED_0201_0603Metric, symbol Device:LED_Small
- removed H1, H2, H3, H4: MountingHole_Pad, NxtPX4:M2MountingHole, symbol Mechanical:MountingHole_Pad
- removed J24: Conn_01x02_Pin, Connector_PinHeader_1.27mm:PinHeader_1x02_P1.27mm_Vertical, symbol Connector:Conn_01x02_Pin
- removed R22: 20kR(0201 9V), Resistor_SMD:R_0201_0603Metric, symbol Device:R_Small
- removed TP12: CAM_9V, NxtPX4:MiniTP, symbol Connector:TestPoint
- removed U11: ICM-20602, NxtPX4:ICM-20602, symbol Sensor_Motion:ICM-20602
- removed U12: HiLAB_Logo, NxtPX4:HILAB_Logo, symbol NxtPX4_Symbol:HiLab-Logo
- removed U15: Signature, NxtPX4:my_signature, symbol NxtPX4_Symbol:Signature
- removed U16: High_temp, NxtPX4:high_temp, symbol NxtPX4_Symbol:High_temperature_Logo
- removed U17: high_voltage, NxtPX4:high_voltage, symbol NxtPX4_Symbol:High_Voltage_Logo
- removed U18: Caution, NxtPX4:Caution, symbol NxtPX4_Symbol:Caution_Logo
- removed U23: MPU6500/ICM20649, NxtPX4:MPU-6500, symbol NxtPX4_Symbol:MPU6500
- removed U5: HKU_Logo, NxtPX4:HKU_Logo, symbol NxtPX4_Symbol:HKU_Logo
- removed U6: UAV_LOGO, NxtPX4:Uav_logo, symbol NxtPX4_Symbol:UAV_LOGO
- removed U7: Direction_Logo, NxtPX4:Direction_Logo, symbol NxtPX4_Symbol:Direction_Logo
- removed U8: RI_LOGO, NxtPX4:Ri_logo, symbol NxtPX4_Symbol:RI_LOGO
- added J3: Conn_02x03_Odd_Even, Connector_PinHeader_1.27mm:PinHeader_2x03_P1.27mm_Vertical_SMD, symbol Connector_Generic:Conn_02x03_Odd_Even
- J25, J26: footprint Connector_PinHeader_1.27mm:PinHeader_1x02_P1.27mm_Vertical -> Connector_PinHeader_1.27mm:PinHeader_1x02_P1.27mm_Vertical_SMD_Pin1Left
Connections:
- net VCC_BAT is gone; now on net VIN: J10.10 (Pin_10)
- net 5V0_SYS: now also J3.1 (Pin_1), J3.3 (Pin_3), J3.5 (Pin_5)
- net at D7.2 (A): now also J3.2 (Pin_2), J3.4 (Pin_4), J3.6 (Pin_6)
- no-connect marks 16 -> 12
Other:
- note removed: "IMU ICM20602 SPI V1.1.0 Design"
- note removed: "Use mounting Holes in order Space to Mount ESC to Carrier"
- moved on the sheet: D7

Commit message: Final PCB version
Other:
- company: HKUST Khalil -> NYU ARPL
- title: NxtPX4 -> Jetson Xavier/Orin NX + PX4 Board
