File: NxtPX4.kicad_sch (KiCad schematic)
At the start: 122 parts, among them J1 USB_C_Receptacle_USB2.0, J10 ESC, J23 Conn_01x04, J24 Micro_SD_Card, J25 Conn_01x02_Pin, J26 Conn_01x02_Pin, J27 GND, J3 Conn_02x03_Odd_Even, J4 ESC, J6 ESC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

Commit message: Made changes to the DHOT, GPS and RC connectors and made them JST 1.25mm. Additionally removed some pins that were deemed unnecessary such as external_heater and buzzer, and made the existing pins more compatible with our GPS and RC.
Parts:
- removed J10, J4: ESC, NxtPX4:01x10_MP_sh1.0_Hori, symbol Connector_Generic_MountingPin:Conn_01x10_MountingPin
- removed J8: UART_Combo, NxtPX4:01x10_MP_sh1.0_Hori, symbol Connector_Generic_MountingPin:Conn_01x10_MountingPin
- removed Q3: SS8050(NPN BEC), Package_TO_SOT_SMD:SOT-23, symbol Device:Q_NPN_BEC
- removed R28: 100R(0201), Resistor_SMD:R_0201_0603Metric, symbol Device:R_Small
- removed R29: 1kR(0201), Resistor_SMD:R_0201_0603Metric, symbol Device:R_Small
- added DSHOT1: ESC, NxtPX4:JST_SM10B-GHS-TB_LF__SN_, symbol Connectors:SM10B-GHS-TB_LF__SN_
- added GPS1: ESC, NxtPX4:JST_SM06B-GHS-TB_LF__SN_, symbol Connectors:SM06B-GHS-TB_LF__SN_
- added RC1: RC, NxtPX4:JST_SM06B-GHS-TB_LF__SN_, symbol Connectors:SM06B-GHS-TB_LF__SN_
- added TP16 (x4): TP, NxtPX4:MiniTP, symbol Connector:TestPoint
Connections:
- net 5V0_SYS: now also GPS1.1, RC1.1
- net BAT_I: now also DSHOT1.7
- net Core_3V3: now also RC1.6
- net GND: now also DSHOT1.9, DSHOT1.S1 (SHIELD), DSHOT1.S2 (SHIELD), GPS1.6, GPS1.S1 (SHIELD), GPS1.S2 (SHIELD), RC1.2, RC1.S1 (SHIELD), RC1.S2 (SHIELD)
- net I2C2_SCL: now also GPS1.4
- net I2C2_SDA: now also GPS1.5
- net PWM/DSHOT_CH1: now also DSHOT1.1
- net PWM/DSHOT_CH2: now also DSHOT1.2
- net PWM/DSHOT_CH3: now also DSHOT1.3
- net PWM/DSHOT_CH4: now also DSHOT1.4
- net PWM/DSHOT_CH5: now also DSHOT1.5, TP16.1
- net PWM/DSHOT_CH6: now also DSHOT1.6, TP16.1
- net SBUS: now also RC1.3
- net UART5_RX: now also RC1.5
- net UART5_TX: now also RC1.4
- net UART7_RX: now also GPS1.2
- net UART7_TX: now also GPS1.3
- net USART3_CK: now also TP16.1
- net USART3_RX: now also DSHOT1.8
- net USART3_TX: now also TP16.1
- net VIN: now also DSHOT1.10
- net AUX_PC0: no longer names the net of U9.F1 (PC0)
- net Buzzer_RGB_LED: no longer names the net of U9.E10 (PC7)
- net Extern_I2C_INT_PE15: no longer names the net of U9.H7 (PE15)
- net Extern_IMU_Heater: no longer names the net of U9.K5 (PE9)
- net Extern_SPI_CS_1_PE13: no longer names the net of U9.K6 (PE13)
- net Extern_SPI_INT_2_PE11: no longer names the net of U9.H6 (PE11)
- no-connect marks 12 -> 18

Commit message: Made a few placement changes for the capacitors, and selected an inductor for the Buck converter
Parts:
- removed DSHOT1: ESC, NxtPX4:JST_SM10B-GHS-TB_LF__SN_, symbol Connectors:SM10B-GHS-TB_LF__SN_
- removed USART_Combo1: UART_Combo, NxtPX4:01x10_MP_sh1.0_Hori, symbol Connector_Generic_MountingPin:Conn_01x10_MountingPin
- added J6: ESC, NxtPX4:01x10_MP_sh1.0_Hori, symbol Connector_Generic_MountingPin:Conn_01x10_MountingPin
- added USARTCombo1: USART Combo, NxtPX4:JST_SM10B-GHS-TB_LF__SN_, symbol Connectors:SM10B-GHS-TB_LF__SN_
Connections:
- net 5V0_SYS: now also USARTCombo1.1, USARTCombo1.6
- net BAT_I: now also J6.7 (Pin_7)
- net GND: now also J6.9 (Pin_9), J6.MP (MountPin), USARTCombo1.2, USARTCombo1.7, USARTCombo1.S1 (SHIELD), USARTCombo1.S2 (SHIELD)
- net PWM/DSHOT_CH1: now also J6.1 (Pin_1)
- net PWM/DSHOT_CH2: now also J6.2 (Pin_2)
- net PWM/DSHOT_CH3: now also J6.3 (Pin_3)
- net PWM/DSHOT_CH4: now also J6.4 (Pin_4)
- net PWM/DSHOT_CH5: now also J6.5 (Pin_5)
- net PWM/DSHOT_CH6: now also J6.6 (Pin_6)
- net USART1_CK: now also USARTCombo1.10
- net USART1_RX: now also USARTCombo1.9
- net USART1_TX: now also USARTCombo1.8
- net USART2_CK: now also USARTCombo1.5
- net USART2_RX: now also USARTCombo1.4
- net USART2_TX: now also USARTCombo1.3
- net USART3_RX: now also J6.8 (Pin_8)
- net VIN: now also J6.10 (Pin_10)
- net USB_OTG_FS_DM renamed USB_OTG_FS_D_N
- net USB_OTG_FS_DP renamed USB_OTG_FS_D_P
