File: csi.kicad_sch (KiCad schematic)
At the start: 38 parts, among them J1 WE_68715014522, J2 WE_68715014022, T1 BSS138APW, U1 PCA9547BS,118

Commit message: Final PCB version
Other:
- company: Antmicro Ltd -> NYU ARPL
- title: Jetson Nano Baseboard -> Jetson Xavier/Orin NX + PX4 Board
