File: display.kicad_sch (KiCad schematic)
At the start: 47 parts, among them IC3 PCA9517ADP, J4 46756-1001, T5 BSS138APW

Commit message: Final PCB version
Other:
- company: Antmicro Ltd -> NYU ARPL
- title: Jetson Nano Baseboard -> Jetson Xavier/Orin NX + PX4 Board
