File: id-serial.kicad_sch (KiCad schematic)
At the start: 5 parts, among them IC1 AT24CS01-ST

Commit message: Final PCB version
Other:
- company: Antmicro Ltd -> NYU ARPL
- title: Jetson Nano Baseboard -> Jetson Xavier/Orin NX + PX4 Board
