File: interfaces.kicad_sch (KiCad schematic)
At the start: 33 parts, among them J10 SI-51005-F, J8 SM04B-SRSS-TB-LF-SN, J9 SM04B-SRSS-TB-LF-SN, U7 MAX3051EKA

Commit message: Final PCB version
Other:
- company: Antmicro Ltd -> NYU ARPL
- title: Jetson Nano Baseboard -> Jetson Xavier/Orin NX + PX4 Board
