File: som.kicad_sch (KiCad schematic)
At the start: 46 parts, among them T2 BSS138APW, T3 BSS138APW, T4 BSS138APW

Commit message: Latest Update
Connections:
- net UART0_RX: no longer M1.203 (UART1_TXD), TP16.1 (P)
- new net UART0_TX: M1.203 (UART1_TXD), TP16.1 (P)
Changed lines of the file:
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@@
   (junction (at 182.88 68.58) (diameter 0) (color 0 0 0 0)
-  )
-  (junction (at 195.58 48.26) (diameter 0) (color 0 0 0 0)
   )
   (junction (at 40.64 48.26) (diameter 0) (color 0 0 0 0)
@@
     (stroke (width 0) (type default))
   )
-  (wire (pts (xy 195.58 48.26) (xy 205.74 48.26))
-    (stroke (width 0) (type default))
-  )
   (wire (pts (xy 294.64 195.58) (xy 292.1 195.58))
     (stroke (width 0) (type default))
@@
     (stroke (width 0) (type default))
   )
-  (wire (pts (xy 190.5 48.26) (xy 195.58 48.26))
-    (stroke (width 0) (type default))
-  )
+  (wire (pts (xy 190.5 48.26) (xy 205.74 48.26))
+    (stroke (width 0) (type default))
+  )

Commit message: Final PCB version
Parts:
- added C79, C80, C81, C85, C89: C_330u_KEMET_B, jetson-nano-baseboard-footprints:0603-cap, symbol jetson-nano-baseboard:C_330u_KEMET_B
- C3, C4: footprint jetson-nano-baseboard-footprints:KEMET_B -> jetson-nano-baseboard-footprints:0603-cap; Val 330u -> 22u/16V
Connections:
- net GND: now also C79.2, C80.2, C81.2, C85.2, C89.2
- net VDD_MOD: now also C79.1, C80.1, C81.1, C85.1, C89.1
Other:
- company: Antmicro Ltd -> NYU ARPL
- title: Jetson Nano Baseboard -> Jetson Xavier/Orin NX + PX4 Board
