File: usb-debug.kicad_sch (KiCad schematic)
At the start: 96 parts, among them IC10 TPS7A0518PDBVT, IC11 NCP380LSNAJAAT1G, IC12 NCP380LSNAJAAT1G, IC7 HD3SS3220, IC9 NCP380LSNAJAAT1G, J12 632723300011, J13 USB_A, T7 BSS138APW, T8 BSS138APW, T9 BSS138APW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

Commit message: Latest Update
Parts:
- J13: footprint Connector_USB:USB_A_TE_292303-7_Horizontal -> Connector_USB:USB_Micro-B_Molex_47346-0001
Changed lines of the file:
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@@
       (effects (font (size 1.27 1.27)))
     )
-    (property "Footprint" "Connector_USB:USB_A_TE_292303-7_Horizontal" (at 389.382 184.912 0)
+    (property "Footprint" "Connector_USB:USB_Micro-B_Molex_47346-0001" (at 389.382 184.912 0)
       (effects (font (size 1.27 1.27)) hide)
     )

Commit message: Final PCB version
Other:
- company: Antmicro Ltd -> NYU ARPL
- title: Jetson Nano Baseboard -> Jetson Xavier/Orin NX + PX4 Board
