File: wifimodule.kicad_sch (KiCad schematic)
At the start: 12 parts, among them J27 Bus_M.2_Socket_E

Commit message: Final PCB version
Other:
- company: (none) -> NYU ARPL
- title: (none) -> Jetson Xavier/Orin NX + PX4 Board
Changed lines of the file:
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@@
 (kicad_sch (version 20230121) (generator eeschema)
   (paper "A4")
+  (title_block
+    (title "Jetson Xavier/Orin NX + PX4 Board")
+    (date "2023-09-28")
+    (rev "1.0")
+    (company "NYU ARPL")
+    (comment 1 "https://wp.nyu.edu/arpl/")
+  )
   (junction (at 233.934 28.448) (diameter 0) (color 0 0 0 0)
   )
@@
     (pin "2")
     (instances
-      (project "V1.1"
+      (project "V1.1_version_control_final"
         (path "/9df9f3e2-e127-4935-b743-4d95c8ce9b2e/9a1170cd-5c8e-46c5-be1f-5e1d7c269927"
           (reference "R170") (unit 1)
@@
     (pin "9")
     (instances
-      (project "V1.1"
+      (project "V1.1_version_control_final"
         (path "/9df9f3e2-e127-4935-b743-4d95c8ce9b2e"
           (reference "J27") (unit 1)
         )
         (path "/9df9f3e2-e127-4935-b743-4d95c8ce9b2e/9a1170cd-5c8e-46c5-be1f-5e1d7c269927"
-          (reference "J27") (unit 1)
+          (reference "Wifi1") (unit 1)
         )
       )
@@
     (pin "2")
     (instances
-      (project "V1.1"
+      (project "V1.1_version_control_final"
         (path "/9df9f3e2-e127-4935-b743-4d95c8ce9b2e/9a1170cd-5c8e-46c5-be1f-5e1d7c269927"
           (reference "R169") (unit 1)
@@
     (pin "2")
     (instances
-      (project "V1.1"
+      (project "V1.1_version_control_final"
         (path "/9df9f3e2-e127-4935-b743-4d95c8ce9b2e/9a1170cd-5c8e-46c5-be1f-5e1d7c269927"
           (reference "R167") (unit 1)
@@
     (pin "2")
     (instances
-      (project "V1.1"
+      (project "V1.1_version_control_final"
         (path "/9df9f3e2-e127-4935-b743-4d95c8ce9b2e/9a1170cd-5c8e-46c5-be1f-5e1d7c269927"
           (reference "C121") (unit 1)
@@
     (pin "1")
     (instances
-      (project "V1.1"
+      (project "V1.1_version_control_final"
         (path "/9df9f3e2-e127-4935-b743-4d95c8ce9b2e/00000000-0000-0000-0000-0000608e1758"
           (reference "#GND_082") (unit 1)
@@
     (pin "2")
     (instances
-      (project "V1.1"
+      (project "V1.1_version_control_final"
         (path "/9df9f3e2-e127-4935-b743-4d95c8ce9b2e/9a1170cd-5c8e-46c5-be1f-5e1d7c269927"
           (reference "R166") (unit 1)
@@
     (pin "2")
     (instances
-      (project "V1.1"
+      (project "V1.1_version_control_final"
         (path "/9df9f3e2-e127-4935-b743-4d95c8ce9b2e/9a1170cd-5c8e-46c5-be1f-5e1d7c269927"
           (reference "D31") (unit 1)
@@
     (pin "2")
     (instances
-      (project "V1.1"
+      (project "V1.1_version_control_final"
         (path "/9df9f3e2-e127-4935-b743-4d95c8ce9b2e/9a1170cd-5c8e-46c5-be1f-5e1d7c269927"
           (reference "D29") (unit 1)
@@
     (pin "1")
     (instances
-      (project "V1.1"
+      (project "V1.1_version_control_final"
         (path "/9df9f3e2-e127-4935-b743-4d95c8ce9b2e/9a1170cd-5c8e-46c5-be1f-5e1d7c269927"
           (reference "#PWR073") (unit 1)
@@
     (pin "2")
     (instances
-      (project "V1.1"
+      (project "V1.1_version_control_final"
         (path "/9df9f3e2-e127-4935-b743-4d95c8ce9b2e/9a1170cd-5c8e-46c5-be1f-5e1d7c269927"
           (reference "C122") (unit 1)
@@
     (pin "2")
     (instances
-      (project "V1.1"
+      (project "V1.1_version_control_final"
         (path "/9df9f3e2-e127-4935-b743-4d95c8ce9b2e/9a1170cd-5c8e-46c5-be1f-5e1d7c269927"
           (reference "R171") (unit 1)
@@
     (pin "1")
     (instances
-      (project "V1.1"
+      (project "V1.1_version_control_final"
         (path "/9df9f3e2-e127-4935-b743-4d95c8ce9b2e/00000000-0000-0000-0000-0000608e1758"
           (reference "SP7") (unit 1)
@@
     (pin "1")
     (instances
-      (project "V1.1"
+      (project "V1.1_version_control_final"
         (path "/9df9f3e2-e127-4935-b743-4d95c8ce9b2e/9a1170cd-5c8e-46c5-be1f-5e1d7c269927"
           (reference "#PWR072") (unit 1)
@@
     (pin "2")
     (instances
-      (project "V1.1"
+      (project "V1.1_version_control_final"
         (path "/9df9f3e2-e127-4935-b743-4d95c8ce9b2e/9a1170cd-5c8e-46c5-be1f-5e1d7c269927"
           (reference "D30") (unit 1)
