File: supply.kicad_sch (KiCad schematic)
At the start: 98 parts, among them IC4 TPS7A0518PDBVT, IC5 74HC00PW, IC6 SN74LVC1G126DCKR, J6 533980471, T6 BSS138APW, U2 LM3671MF-3.3/NOPB, U3 LM3671MF-3.3/NOPB, U4 LM62440-Q1, U5 SIC477ED-T1-GE3, U6 SN74LXC1T45DBVR

Commit message: Latest Update
Parts:
- J5: value ~ -> DC_SOCKET
Changed lines of the file:
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@@
   (junction (at 341.63 62.23) (diameter 0) (color 0 0 0 0)
   )
-  (junction (at 231.14 257.81) (diameter 0) (color 0 0 0 0)
-  )
   (junction (at 62.23 53.34) (diameter 0) (color 0 0 0 0)
   )
@@
   (junction (at 160.02 160.02) (diameter 0) (color 0 0 0 0)
   )
+  (junction (at 217.424 256.667) (diameter 0) (color 0 0 0 0)
+  )
   (junction (at 80.01 81.28) (diameter 0) (color 0 0 0 0)
   )
@@
     (stroke (width 0) (type default))
   )
-  (wire (pts (xy 231.14 255.27) (xy 228.6 255.27))
-    (stroke (width 0) (type default))
-  )
   (wire (pts (xy 152.4 77.47) (xy 161.29 77.47))
     (stroke (width 0) (type default))
@@
     (stroke (width 0) (type default))
   )
+  (wire (pts (xy 219.71 252.73) (xy 231.14 252.73))
+    (stroke (width 0) (type default))
+  )
   (wire (pts (xy 31.75 53.34) (xy 34.29 53.34))
     (stroke (width 0) (type default))
@@
     (stroke (width 0) (type default))
   )
+  (wire (pts (xy 213.614 259.207) (xy 217.424 259.207))
+    (stroke (width 0) (type default))
+  )
   (wire (pts (xy 93.98 190.5) (xy 102.87 190.5))
     (stroke (width 0) (type default))
@@
     (stroke (width 0) (type default))
   )
+  (wire (pts (xy 217.424 256.667) (xy 231.14 256.667))
+    (stroke (width 0) (type default))
+  )
   (wire (pts (xy 160.02 152.4) (xy 160.02 160.02))
     (stroke (width 0) (type default))
@@
     (stroke (width 0) (type default))
   )
-  (wire (pts (xy 231.14 257.81) (xy 228.6 257.81))
-    (stroke (width 0) (type default))
-  )
   (wire (pts (xy 341.63 46.99) (xy 335.28 46.99))
     (stroke (width 0) (type default))
@@
     (stroke (width 0) (type default))
   )
+  (wire (pts (xy 219.71 252.73) (xy 219.71 254.127))
+    (stroke (width 0) (type default))
+  )
   (wire (pts (xy 148.59 144.78) (xy 151.13 144.78))
     (stroke (width 0) (type default))
@@
     (stroke (width 0) (type default))
   )
-  (wire (pts (xy 231.14 257.81) (xy 231.14 255.27))
-    (stroke (width 0) (type default))
-  )
   (wire (pts (xy 119.38 190.5) (xy 118.11 190.5))
     (stroke (width 0) (type default))
@@
     (stroke (width 0) (type default))
   )
-  (wire (pts (xy 231.14 252.73) (xy 228.6 252.73))
-    (stroke (width 0) (type default))
-  )
   (wire (pts (xy 280.67 85.09) (xy 279.4 85.09))
     (stroke (width 0) (type default))
@@
     (stroke (width 0) (type default))
   )
+  (wire (pts (xy 217.424 259.207) (xy 217.424 256.667))
+    (stroke (width 0) (type default))
+  )
   (wire (pts (xy 341.63 80.01) (xy 341.63 85.09))
     (stroke (width 0) (type default))
@@
     (stroke (width 0) (type default))
   )
+  (wire (pts (xy 213.614 254.127) (xy 219.71 254.127))
+    (stroke (width 0) (type default))
+  )
   (wire (pts (xy 182.88 68.58) (xy 182.88 73.66))
     (stroke (width 0) (type default))
@@
     (stroke (width 0) (type default))
   )
+  (wire (pts (xy 213.614 256.667) (xy 217.424 256.667))
+    (stroke (width 0) (type default))
+  )
   (wire (pts (xy 341.63 72.39) (xy 341.63 67.31))
     (stroke (width 0) (type default))
@@
     (stroke (width 0) (type default))
   )
-  (wire (pts (xy 231.14 257.81) (xy 231.14 264.16))
+  (wire (pts (xy 231.14 256.667) (xy 231.14 264.16))
     (stroke (width 0) (type default))
   )
@@
     )
   )
-  (symbol (lib_id "jetson-nano-baseboard:DC_SOCKET") (at 223.52 255.27 0) (unit 1)
-    (in_bom yes) (on_board yes) (dnp no)
-    (property "Reference" "J5" (at 214.63 261.112 0)
-      (effects (font (size 1.524 1.524)) (justify left bottom))
-    )
-    (property "Value" "~" (at 223.52 255.27 0)
-      (effects (font (size 1.27 1.27)) hide)
-    )
-    (property "Footprint" "jetson-nano-baseboard-footprints:DC_SOCKET" (at 223.52 255.27 0)
-      (effects (font (size 1.27 1.27)) hide)
-    )
-    (property "Datasheet" "" (at 223.52 255.27 0)
-      (effects (font (size 1.27 1.27)) hide)
-    )
-    (property "MPN" "MJ-179PH" (at 136.4234 664.5148 0)
-      (effects (font (size 1.27 1.27)) hide)
-    )
-    (property "Manufacturer" "Multicomp" (at 136.4234 664.5148 0)
-      (effects (font (size 1.27 1.27)) hide)
-    )
-    (pin "1")
-    (pin "2")
-    (pin "3")
-    (instances
-      (project "V1.1"
-        (path "/9df9f3e2-e127-4935-b743-4d95c8ce9b2e/00000000-0000-0000-0000-0000608dc6e9"
-          (reference "J5") (unit 1)
-        )
-      )
-    )
-  )
   (symbol (lib_id "jetson-nano-baseboard:SN74LVC1G126") (at 364.49 67.31 0) (unit 1)
     (in_bom yes) (on_board yes) (dnp no)
@@
         )
       )
+    )
+  )
+  (symbol (lib_id "jetson-nano-baseboard:DC_SOCKET") (at 208.534 256.667 0) (unit 1)
+    (in_bom yes) (on_board yes) (dnp no)
+    (property "Reference" "J5" (at 204.597 250.952 0)
+      (effects (font (size 1.524 1.524)))
+    )
+    (property "Value" "DC_SOCKET" (at 208.534 256.667 0)
+      (effects (font (size 1.524 1.524)) hide)
+    )
+    (property "Footprint" "jetson-nano-baseboard-footprints:DC_SOCKET" (at 208.534 256.667 0)
+      (effects (font (size 1.524 1.524)) hide)
+    )
+    (property "Datasheet" "" (at 208.534 256.667 0)
+      (effects (font (size 1.524 1.524)) hide)
+    )
+    (property "Manufacturer" "Multicomp" (at 208.534 256.667 0)
+      (effects (font (size 1.27 1.27)) hide)
+    )
+    (property "MPN" "MJ-179PH" (at 208.534 256.667 0)
+      (effects (font (size 1.27 1.27)) hide)
+    )
+    (pin "1")
+    (pin "2")
+    (pin "3")
+    (instances
+      (project "V1.1"
+        (path "/9df9f3e2-e127-4935-b743-4d95c8ce9b2e/00000000-0000-0000-0000-0000608dc6e9"
+          (reference "J5") (unit 1)
+        )
+      )

Commit message: Final PCB version
Parts:
- removed J5: DC_SOCKET, jetson-nano-baseboard-footprints:DC_SOCKET, symbol jetson-nano-baseboard:DC_SOCKET
- added C123, C98: C_47u_0805, jetson-nano-baseboard-footprints:0603-cap, symbol jetson-nano-baseboard:C_47u_0805
- added C96: C_10u_1206_50V, jetson-nano-baseboard-footprints:1206-cap, symbol jetson-nano-baseboard:C_10u_1206_50V
- added U9: XT30UPB-M, jetson-nano-baseboard-footprints:XT30UPB-M, symbol XT30PW-M:XT30UPB-M
- C22: Val 10u/50V -> 22u/50V
- C24: Val 10u/50V -> 100u/50V
- C31: footprint jetson-nano-baseboard-footprints:0805-cap -> jetson-nano-baseboard-footprints:0603-cap; Val 10u -> 22u/16V
- C36: footprint jetson-nano-baseboard-footprints:0805-cap -> jetson-nano-baseboard-footprints:0603-cap; Val 47u -> 22u/16V
- U4: value LM62440-Q1 -> LM61460-Q1
- U5: value SIC477ED-T1-GE3 -> SIC476ED-T1-GE3; MPN SIC477ED-T1-GE3 -> SIC476ED-T1-GE3
Connections:
- net 3V3_SYS: now also C123.1, C98.1
- net 3V3_VIN: now also C96.1
- net GND: now also C123.2, C96.2, C98.2, U9.P$2 (-)
- net at F3.1: now also U9.P$1 (+)
Other:
- note added: "5V/12A"
- note removed: "5V/8A"
- company: Antmicro Ltd -> NYU ARPL
- title: Jetson Nano Baseboard -> Jetson Xavier/Orin NX + PX4 Board

Commit message: Made a few placement changes for the capacitors, and selected an inductor for the Buck converter
Parts:
- L6: value IHLP3232DZER3R3M01 -> IHLP3232DZER2R2M01; Val 3u3/9.2A -> 2u2/10.5 A
Changed lines of the file:
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@@
       (effects (font (size 1.524 1.524)))
     )
-    (property "Value" "IHLP3232DZER3R3M01" (at 167.64 58.42 0)
+    (property "Value" "\nIHLP3232DZER2R2M01" (at 167.64 58.42 0)
       (effects (font (size 1.524 1.524)))
     )
@@
       (effects (font (size 1.27 1.27)) hide)
     )
-    (property "Val" "3u3/9.2A" (at 167.64 62.23 0)
+    (property "Val" "2u2/10.5 A" (at 167.64 62.23 0)
       (effects (font (size 1.27 1.27)))
     )
